File: schematics/Orion68/orion68io.kicad_sch (KiCad schematic)
At the start: 41 parts, among them J1 LevelConverter, J200 Euro96pin, J22 Kbd_usb, J23 RTC, J26 DuartB, J28 DuartA, Q4 3.6864MHz, U16 74HC138, U21 74HC4078, U22 74LS08, U25 SN74LVC245APW, U26 SN74LVC245APW, U30 LM2937xT, U33 68681, U36 UART2, U43 74HC4078, U44 74HC138

Commit message: 2026/10/27:(A) added A10 to pin11 74HC4078
Connections:
- net A10: now also U43.11 (I7)
- net GND: no longer U43.11 (I7)
Changed lines of the file:
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@@
 	)
 	(junction
-		(at 26.67 196.85)
-		(diameter 0)
-		(color 0 0 0 0)
-	)
-	(junction
 		(at -10.795 249.555)
 		(diameter 0)
@@
 	(wire
 		(pts
-			(xy 29.845 194.31) (xy 30.48 194.945)
-		)
-		(stroke
-			(width 0)
-			(type default)
-		)
-	)
-	(wire
-		(pts
 			(xy 160.02 92.71) (xy 160.02 95.25)
 		)
@@
 	(wire
 		(pts
-			(xy 26.67 194.31) (xy 26.67 196.85)
-		)
-		(stroke
-			(width 0)
-			(type default)
-		)
-	)
-	(wire
-		(pts
 			(xy 212.09 154.94) (xy 212.09 157.48)
 		)
@@
 		)
 	)
-	(wire
-		(pts
-			(xy 26.67 194.31) (xy 29.845 194.31)
-		)
-		(stroke
-			(width 0)
-			(type default)
-		)
-	)
 	(polyline
 		(pts
@@
 		(effects
 			(font
+				(size 1.27 1.27)
+			)
+			(justify right bottom)
+		)
+	)
+	(label "A10"
+		(at 30.48 194.945 180)
+		(effects
+			(font
